Commit message: gripper in rviz, but wrong orientation

File: src/khi_robot/khi_duaro_description/urdf/duaro.urdf.xacro (robot description, xacro)
@@ -1,14 +1,22 @@
 <?xml version="1.0" ?>
 <robot name="khi_duaro" xmlns:xacro="http://ros.org/wiki/xacro">
+  <xacro:arg name="prefix" default="duaro" />
   <xacro:include filename="$(find khi_duaro_description)/urdf/duaro_macro.xacro"/>
+  <xacro:include filename="$(find khi_duaro_description)/urdf/wsg_50.urdf.xacro"/>
   <!-- instantiate duaro -->
-  <xacro:khi_duaro prefix="" />
-  <xacro:include filename="$(find wsg_50_simulation)/urdf/wsg_50.urdf"/>
-  <xacro:wsg_50_xacro prefix="" />
+  <xacro:khi_duaro prefix="$(arg prefix)" />
+  <!-- lower gripper -->
+  <xacro:wsg_50_xacro name="lower_gripper" parent="$(arg prefix)lower_link_j4" finger_length="0.023" finger_tip="0">
+    <origin xyz="0 0 0" rpy="0 0 0" />
+  </xacro:wsg_50_xacro>
+  <!-- upper gripper-->
+  <xacro:wsg_50_xacro name="upper_gripper" parent="$(arg prefix)upper_link_j4" finger_length="0.023" finger_tip="0">
+    <origin xyz="0 0 0" rpy="0 0 0" />
+  </xacro:wsg_50_xacro>
   <!-- Fix duaro to world -->
   <link name="world"/>
   <joint name="world2base" type="fixed">
     <parent link="world"/>
-    <child link="base_link"/>
+    <child link="$(arg prefix)base_link"/>
     <origin rpy="0 0 0" xyz="0 0 0"/>
   </joint>
