Commit message: Correct gripper orientation

File: src/khi_robot/khi_duaro_description/urdf/wsg_50.urdf.xacro (robot description, xacro)
@@ -25,5 +25,5 @@
       </inertial>
       <visual>
-          <origin xyz="0.0 0 0" rpy="0 0 0" />
+          <origin xyz="0.0 0 0" rpy="3.14 0 0" />
           <geometry>
              <mesh filename="package://wsg_50_simulation/meshes/WSG50_110.stl" scale="1 1 1"/>
@@ -35,5 +35,5 @@
       </visual>
       <collision>
-          <origin xyz="0.0 0 0" rpy="0 0 0" />
+          <origin xyz="0.0 0 0" rpy="3.14 0 0" />
           <geometry>
 	     <!--box size="0.146 0.05 0.0735"/-->
@@ -78,15 +78,15 @@
       </inertial>
       <visual>
-          <origin xyz="0.0 0 0" rpy="0 0 0" />
-          <geometry>
-             <mesh filename="package://wsg_50_simulation/meshes/GUIDE_WSG50_110.stl" scale="0.001 0.001 0.001"/>
-	     <!--box size="0.0175 0.03 0.024"/-->
-          </geometry>
-          <material name="black">
-		<color rgba="0 0 0 0"/>
-      	  </material>
-      </visual>
-      <collision>
-          <origin xyz="0 0 0" rpy="0 0 0" />
+          <origin xyz="0.0 0 0" rpy="3.14 0 0" />
+          <geometry>
+             <mesh filename="package://wsg_50_simulation/meshes/GUIDE_WSG50_110.stl" scale="0.001 0.001 0.001"/>
+	     <!--box size="0.0175 0.03 0.024"/-->
+          </geometry>
+          <material name="black">
+		<color rgba="0 0 0 1"/>
+      	  </material>
+      </visual>
+      <collision>
+          <origin xyz="0 0 0" rpy="3.14 0 0" />
           <geometry>
 	     <!--box size="0.0175 0.03 0.024"/-->
@@ -118,14 +118,14 @@
       </inertial>
       <visual>
-          <origin xyz="0.0 0 0" rpy="0 0 0" />
-          <geometry>
-             <mesh filename="package://wsg_50_simulation/meshes/WSG-FMF.stl" scale="0.001 0.001 0.001"/>
-          </geometry>
-          <material name="black">
-		<color rgba="0 0 0 0"/>
-      	  </material>
-      </visual>
-      <collision>
-          <origin xyz="0 0 0" rpy="0 0 0" />
+          <origin xyz="0.0 0 0" rpy="3.14 0 0" />
+          <geometry>
+             <mesh filename="package://wsg_50_simulation/meshes/WSG-FMF.stl" scale="0.001 0.001 0.001"/>
+          </geometry>
+          <material name="black">
+		<color rgba="0 0 0 1"/>
+      	  </material>
+      </visual>
+      <collision>
+          <origin xyz="0 0 0" rpy="3.14 0 0" />
           <geometry>
              <mesh filename="package://wsg_50_simulation/meshes/WSG-FMF.stl" scale="0.001 0.001 0.001"/>
@@ -163,15 +163,15 @@
       </inertial>
       <visual>
-          <origin xyz="0.0 0 0" rpy="0 0 0" />
-          <geometry>
-             <mesh filename="package://wsg_50_simulation/meshes/GUIDE_WSG50_110.stl" scale="0.001 0.001 0.001"/>
-	     <!--box size="0.0175 0.03 0.024"/-->
-          </geometry>
-          <material name="black">
-		<color rgba="0 0 0 0"/>
-      	  </material>
-      </visual>
-      <collision>
-          <origin xyz="0 0 0" rpy="0 0 0" />
+          <origin xyz="0.0 0 0" rpy="3.14 0 0" />
+          <geometry>
+             <mesh filename="package://wsg_50_simulation/meshes/GUIDE_WSG50_110.stl" scale="0.001 0.001 0.001"/>
+	     <!--box size="0.0175 0.03 0.024"/-->
+          </geometry>
+          <material name="black">
+		<color rgba="0 0 0 1"/>
+      	  </material>
+      </visual>
+      <collision>
+          <origin xyz="0 0 0" rpy="3.14 0 0" />
           <geometry>
 	     <!--box size="0.0175 0.03 0.024"/-->
@@ -203,14 +203,14 @@
       </inertial>
       <visual>
-          <origin xyz="0.0 0 0" rpy="0 0 0" />
-          <geometry>
-             <mesh filename="package://wsg_50_simulation/meshes/WSG-FMF.stl" scale="0.001 0.001 0.001"/>
-          </geometry>
-          <material name="black">
-		<color rgba="0 0 0 0"/>
-      	  </material>
-      </visual>
-      <collision>
-          <origin xyz="0 0 0" rpy="0 0 0" />
+          <origin xyz="0.0 0 0" rpy="3.14 0 0" />
+          <geometry>
+             <mesh filename="package://wsg_50_simulation/meshes/WSG-FMF.stl" scale="0.001 0.001 0.001"/>
+          </geometry>
+          <material name="black">
+		<color rgba="0 0 0 1"/>
+      	  </material>
+      </visual>
+      <collision>
+          <origin xyz="0 0 0" rpy="3.14 0 0" />
           <geometry>
              <mesh filename="package://wsg_50_simulation/meshes/WSG-FMF.stl" scale="0.001 0.001 0.001"/>
