Commit message: Grippers added and functional

File: Unity_env/Assets/URDF/duaro.urdf (robot description, URDF)
Before this commit: robot khi_duaro, 19 links, 18 joints
Links:
- removed link base_link
- removed link cart
- removed link duaro_body
- removed link duaro_body_cover
- removed link duaro_j0
- removed link duaro_j0_cover
- removed link duaro_logo
- removed link kawasaki_logo
- removed link lower_link_j1
- removed link lower_link_j2
- removed link lower_link_j3
- removed link lower_link_j3_obst
- removed link lower_link_j4
- removed link upper_link_j1
- removed link upper_link_j2
- removed link upper_link_j3
- removed link upper_link_j3_obst
- removed link upper_link_j4
- added link duarobase_link; collision mesh filename=package://khi_duaro_description/meshes/WD002N_F502_Adjuster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; visual mesh filename=package://khi_duaro_description/meshes/WD002N_F502_Adjuster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
- added link duarocart, mass 2; collision mesh filename=package://khi_duaro_description/meshes/WD002N_F502_Cart.stl; visual mesh filename=package://khi_duaro_description/meshes/WD002N_F502_Cart.stl
- added link duaroduaro_body, mass 100; collision mesh filename=package://khi_duaro_description/meshes/WD002N_F502_Cabinet_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; visual mesh filename=package://khi_duaro_description/meshes/WD002N_F502_Cabinet_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
- added link duaroduaro_body_cover, mass 1; collision mesh filename=package://khi_duaro_description/meshes/WD002N_F502_Cabinet_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; visual mesh filename=package://khi_duaro_description/meshes/WD002N_F502_Cabinet_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
- added link duaroduaro_j0, mass 10; collision mesh filename=package://khi_duaro_description/meshes/WD002N_A201_j0_Ver2m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; visual mesh filename=package://khi_duaro_description/meshes/WD002N_A201_j0_Ver2m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
- added link duaroduaro_j0_cover, mass 2; collision mesh filename=package://khi_duaro_description/meshes/WD002N_A201_j0_cover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; visual mesh filename=package://khi_duaro_description/meshes/WD002N_A201_j0_cover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
- added link duaroduaro_logo, mass 1; collision mesh filename=package://khi_duaro_description/meshes/WD002N_F502_LOGO_duA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; visual mesh filename=package://khi_duaro_description/meshes/WD002N_F502_LOGO_duA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
- added link duarokawasaki_logo, mass 1; collision mesh filename=package://khi_duaro_description/meshes/WD002N_F502_LOGO_Kaw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; visual mesh filename=package://khi_duaro_description/meshes/WD002N_F502_LOGO_Kaw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
- added link duarolower_link_j1, mass 11.463; collision mesh filename=package://khi_duaro_description/meshes/WD002N_A201L_J1_Ver2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; visual mesh filename=package://khi_duaro_description/meshes/WD002N_A201L_J1_Ver2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
- added link duarolower_link_j2, mass 3.747; collision mesh filename=package://khi_duaro_description/meshes/WD002N_A202L_J2m.stl; visual mesh filename=package://khi_duaro_description/meshes/WD002N_A202L_J2m.stl
- added link duarolower_link_j3, mass 3.476; collision mesh filename=package://khi_duaro_description/meshes/WD002N_A202L_J3m.stl; visual mesh filename=package://khi_duaro_description/meshes/WD002N_A202L_J3m.stl
- added link duarolower_link_j3_obst; visual mesh filename=package://khi_duaro_description/meshes/WD002N_A202L_J3_obst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
- added link duarolower_link_j4, mass 0.5; collision mesh filename=package://khi_duaro_description/meshes/WD002N_A202L_J4m.stl; visual mesh filename=package://khi_duaro_description/meshes/WD002N_A202L_J4m.stl
- added link duaroupper_link_j1, mass 11.452; collision mesh filename=package://khi_duaro_description/meshes/WD002N_A201U_J1_Ver2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; visual mesh filename=package://khi_duaro_description/meshes/WD002N_A201U_J1_Ver2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
- added link duaroupper_link_j2, mass 3.751; collision mesh filename=package://khi_duaro_description/meshes/WD002N_A202U_J2m.stl; visual mesh filename=package://khi_duaro_description/meshes/WD002N_A202U_J2m.stl
- added link duaroupper_link_j3, mass 3.476; collision mesh filename=package://khi_duaro_description/meshes/WD002N_A202U_J3m.stl; visual mesh filename=package://khi_duaro_description/meshes/WD002N_A202U_J3m.stl
- added link duaroupper_link_j3_obst; visual mesh filename=package://khi_duaro_description/meshes/WD002N_A202U_J3_obst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
- added link duaroupper_link_j4, mass 10; collision mesh filename=package://khi_duaro_description/meshes/WD002N_A202U_J4m.stl; visual mesh filename=package://khi_duaro_description/meshes/WD002N_A202U_J4m.stl
- added link lower_gripper_base_link, mass 0.25; collision mesh filename=package://wsg_50_simulation/meshes/WSG50_110.stl scale=1 1 1; visual mesh filename=package://wsg_50_simulation/meshes/WSG50_110.stl scale=1 1 1
- added link lower_gripper_center
- added link lower_gripper_finger_left, mass 0.1; collision mesh filename=package://wsg_50_simulation/meshes/WSG-FMF.stl scale=0.001 0.001 0.001; visual mesh filename=package://wsg_50_simulation/meshes/WSG-FMF.stl scale=0.001 0.001 0.001
- added link lower_gripper_finger_right, mass 0.1; collision mesh filename=package://wsg_50_simulation/meshes/WSG-FMF.stl scale=0.001 0.001 0.001; visual mesh filename=package://wsg_50_simulation/meshes/WSG-FMF.stl scale=0.001 0.001 0.001
- added link lower_gripper_gripper_left, mass 0.1; collision mesh filename=package://wsg_50_simulation/meshes/GUIDE_WSG50_110.stl scale=0.001 0.001 0.001; visual mesh filename=package://wsg_50_simulation/meshes/GUIDE_WSG50_110.stl scale=0.001 0.001 0.001
- added link lower_gripper_gripper_right, mass 0.1; collision mesh filename=package://wsg_50_simulation/meshes/GUIDE_WSG50_110.stl scale=0.001 0.001 0.001; visual mesh filename=package://wsg_50_simulation/meshes/GUIDE_WSG50_110.stl scale=0.001 0.001 0.001
- added link upper_gripper_base_link, mass 0.25; collision mesh filename=package://wsg_50_simulation/meshes/WSG50_110.stl scale=1 1 1; visual mesh filename=package://wsg_50_simulation/meshes/WSG50_110.stl scale=1 1 1
- added link upper_gripper_center
- added link upper_gripper_finger_left, mass 0.1; collision mesh filename=package://wsg_50_simulation/meshes/WSG-FMF.stl scale=0.001 0.001 0.001; visual mesh filename=package://wsg_50_simulation/meshes/WSG-FMF.stl scale=0.001 0.001 0.001
- added link upper_gripper_finger_right, mass 0.1; collision mesh filename=package://wsg_50_simulation/meshes/WSG-FMF.stl scale=0.001 0.001 0.001; visual mesh filename=package://wsg_50_simulation/meshes/WSG-FMF.stl scale=0.001 0.001 0.001
- added link upper_gripper_gripper_left, mass 0.1; collision mesh filename=package://wsg_50_simulation/meshes/GUIDE_WSG50_110.stl scale=0.001 0.001 0.001; visual mesh filename=package://wsg_50_simulation/meshes/GUIDE_WSG50_110.stl scale=0.001 0.001 0.001
- added link upper_gripper_gripper_right, mass 0.1; collision mesh filename=package://wsg_50_simulation/meshes/GUIDE_WSG50_110.stl scale=0.001 0.001 0.001; visual mesh filename=package://wsg_50_simulation/meshes/GUIDE_WSG50_110.stl scale=0.001 0.001 0.001
Joints:
- removed joint cart_joint
- removed joint duaro_body_cover_joint
- removed joint duaro_body_joint
- removed joint duaro_j0_cover_joint
- removed joint duaro_logo_joint
- removed joint joint0
- removed joint kawasaki_logo_joint
- removed joint lower_j3_obstaclem_joint
- removed joint lower_joint1
- removed joint lower_joint2
- removed joint lower_joint3
- removed joint lower_joint4
- removed joint upper_j3_obstaclem_joint
- removed joint upper_joint1
- removed joint upper_joint2
- removed joint upper_joint3
- removed joint upper_joint4
- added joint duarocart_joint: type fixed, parent duarobase_link, child duarocart, origin xyz=0 0 0 rpy=0 0 0
- added joint duaroduaro_body_cover_joint: type fixed, parent duarobase_link, child duaroduaro_body_cover, origin xyz=0 0 0 rpy=0 0 0
- added joint duaroduaro_body_joint: type fixed, parent duarobase_link, child duaroduaro_body, origin xyz=0 0 0 rpy=0 0 0
- added joint duaroduaro_j0_cover_joint: type fixed, parent duarobase_link, child duaroduaro_j0_cover, origin xyz=0 0 0.82 rpy=0 0 0
- added joint duaroduaro_logo_joint: type fixed, parent duarobase_link, child duaroduaro_logo, origin xyz=0 0 0 rpy=0 0 0
- added joint duarojoint0: type fixed, parent duaroduaro_body, child duaroduaro_j0, origin xyz=0 0 0.82
- added joint duarokawasaki_logo_joint: type fixed, parent duarobase_link, child duarokawasaki_logo, origin xyz=0 0 0 rpy=0 0 0
- added joint duarolower_j3_obstaclem_joint: type fixed, parent duarolower_link_j3, child duarolower_link_j3_obst, origin xyz=0 0 0 rpy=0 0 0
- added joint duarolower_joint1: type revolute, parent duaroduaro_j0, child duarolower_link_j1, origin xyz=0 0 0.2515 rpy=0 0 0, axis 0 0 1, limit lower=-2.9670597283903604 upper=2.9670597283903604 effort=100.0 velocity=4.1887902047863905
- added joint duarolower_joint2: type revolute, parent duarolower_link_j1, child duarolower_link_j2, origin xyz=0 0.36 0.0905, axis 0 0 1, limit lower=-2.443460952792061 upper=2.443460952792061 effort=100.0 velocity=5.497787143782138
- added joint duarolower_joint3: type prismatic, parent duarolower_link_j2, child duarolower_link_j3, origin xyz=0 0.4 0.03850, axis 0 0 1, limit lower=0 upper=0.15 effort=100.0 velocity=0.3
- added joint duarolower_joint4: type revolute, parent duarolower_link_j3, child duarolower_link_j4, origin xyz=0 0 -0.24, axis 0 0 1, limit lower=-6.283185307179586 upper=6.283185307179586 effort=100.0 velocity=10.471975511965978
- added joint duaroupper_j3_obstaclem_joint: type fixed, parent duaroupper_link_j3, child duaroupper_link_j3_obst, origin xyz=0 0 0
- added joint duaroupper_joint1: type revolute, parent duaroduaro_j0, child duaroupper_link_j1, origin xyz=0 0 0.3805 rpy=0 0 0, axis 0 0 1, limit lower=-2.443460952792061 upper=8.726646259971648 effort=100.0 velocity=4.1887902047863905
- added joint duaroupper_joint2: type revolute, parent duaroupper_link_j1, child duaroupper_link_j2, origin xyz=0 0.36 0, axis 0 0 1, limit lower=-2.443460952792061 upper=2.443460952792061 effort=100.0 velocity=5.497787143782138
- added joint duaroupper_joint3: type prismatic, parent duaroupper_link_j2, child duaroupper_link_j3, origin xyz=0 0.4 0, axis 0 0 1, limit lower=0 upper=0.15 effort=100.0 velocity=0.3
- added joint duaroupper_joint4: type revolute, parent duaroupper_link_j3, child duaroupper_link_j4, origin xyz=0 0 -0.24, axis 0 0 1, limit lower=-6.283185307179586 upper=6.283185307179586 effort=100.0 velocity=0.3
- added joint lower_gripper_anterior_gripper_joint: type fixed, parent duarolower_link_j4, child lower_gripper_base_link
- added joint lower_gripper_center_joint: type fixed, parent lower_gripper_base_link, child lower_gripper_center, origin xyz=0 0 -0.017 rpy=0 0 0
- added joint lower_gripper_finger_left_joint: type prismatic, parent lower_gripper_base_link, child lower_gripper_gripper_left, origin xyz=0 0 0 rpy=0 0 0, axis 1 0 0, limit lower=-0.055 upper=-0.0027 effort=1.0 velocity=1.0
- added joint lower_gripper_finger_right_joint: type prismatic, parent lower_gripper_base_link, child lower_gripper_gripper_right, origin xyz=0 0 0 rpy=0 0 3.14159, axis -1 0 0, limit lower=0.0027 upper=0.055 effort=1.0 velocity=1.0
- added joint lower_gripper_guide_joint_finger_left: type fixed, parent lower_gripper_gripper_left, child lower_gripper_finger_left, origin xyz=0 0 -0.017 rpy=0 0 0, axis 1 0 0, limit effort=100 velocity=100
- added joint lower_gripper_guide_joint_finger_right: type fixed, parent lower_gripper_gripper_right, child lower_gripper_finger_right, origin xyz=0 0 -0.017 rpy=0 0 0, axis 1 0 0, limit effort=100 velocity=100
- added joint upper_gripper_anterior_gripper_joint: type fixed, parent duaroupper_link_j4, child upper_gripper_base_link
- added joint upper_gripper_center_joint: type fixed, parent upper_gripper_base_link, child upper_gripper_center, origin xyz=0 0 -0.017 rpy=0 0 0
- added joint upper_gripper_finger_left_joint: type prismatic, parent upper_gripper_base_link, child upper_gripper_gripper_left, origin xyz=0 0 0 rpy=0 0 0, axis 1 0 0, limit lower=-0.055 upper=-0.0027 effort=1.0 velocity=1.0
- added joint upper_gripper_finger_right_joint: type prismatic, parent upper_gripper_base_link, child upper_gripper_gripper_right, origin xyz=0 0 0 rpy=0 0 3.14159, axis -1 0 0, limit lower=0.0027 upper=0.055 effort=1.0 velocity=1.0
- added joint upper_gripper_guide_joint_finger_left: type fixed, parent upper_gripper_gripper_left, child upper_gripper_finger_left, origin xyz=0 0 -0.017 rpy=0 0 0, axis 1 0 0, limit effort=100 velocity=100
- added joint upper_gripper_guide_joint_finger_right: type fixed, parent upper_gripper_gripper_right, child upper_gripper_finger_right, origin xyz=0 0 -0.017 rpy=0 0 0, axis 1 0 0, limit effort=100 velocity=100
- joint world2base: child base_link -> duarobase_link
